Commit message: update the robot values (core)

File: src/lidar_robot/description/robot_core.xacro (robot description, xacro)
@@ -100,5 +100,5 @@
         <visual>
             <geometry>
-                <sphere radius = "0.05"/>
+                <sphere radius = "0.1"/>
             </geometry>
             <material name = "orange"/>
@@ -106,8 +106,8 @@
         <collision>
             <geometry>
-                <sphere radius = "0.05"/>
+                <sphere radius = "0.1"/>
             </geometry>
         </collision>
-        <xacro:inertial_sphere mass="0.2" radius="0.05">
+        <xacro:inertial_sphere mass="0.2" radius="0.1">
             <origin xyz="0 0 0" rpy="0 0 0" />
         </xacro:inertial_sphere>
