Commit message: added 4 wheel robot and made it run ( diff drive plugin)

File: src/lidar_robot/description/robot.urdf.xacro (robot description, xacro)
@@ -4,3 +4,4 @@
     <!-- <link name="base_link"></link> -->
     <xacro:include filename="robot_core.xacro" />
+    <xacro:include filename="gazebo_robot_control.xacro"/>
 </robot>

File: src/lidar_robot/description/robot_core.xacro (robot description, xacro)
@@ -12,73 +12,50 @@
         <color rgba="0.5 0.5 0.5 1"/>
     </material>
-    <material name = "blue">
+    <material name="blue">
         <color rgba="0.2 0.2 1 1"/>
     </material>
-    <material name = "orange">
-        <color rgba = "1 0.3 0.1 1"/>
+    <material name="orange">
+        <color rgba="1 0.3 0.1 1"/>
     </material>
     <!-- first link is called as base link -->
-    <link name = "base link">
+    <link name="base link">
     </link>
-    <!-- chassis (box with some dimentions) -->
-    <joint name = "chassis_joint" type = "fixed">
-        <parent link = "base link"/>
-        <child link = "chassis"/>
-        <origin xyz = "-0.1 0 0"/>
+    <!-- chassis (box with some dimensions) -->
+    <joint name="chassis_joint" type="fixed">
+        <parent link="base link"/>
+        <child link="chassis"/>
+        <origin xyz="-0.1 0 0"/>
     </joint>
-    <link name = "chassis">
+    <link name="chassis">
         <visual>
-            <origin xyz = "0.2 0 0.1" />
+            <origin xyz="0.2 0 0.1" />
             <geometry>
-                <box size = "0.4 0.3 0.2"/>
+                <box size="0.4 0.3 0.2"/>
             </geometry>
-            <material name = "grey"/>
+            <material name="grey"/>
         </visual>
         <collision>
-            <origin xyz = "0.2 0 0.1" />
+            <origin xyz="0.2 0 0.1" />
             <geometry>
-                <box size = "0.4 0.3 0.2"/>
+                <box size="0.4 0.3 0.2"/>
             </geometry>
         </collision>
-        <xacro:inertial_box mass = "0.5" x="0.4" y="0.3" z="0.2">
+        <xacro:inertial_box mass="0.5" x="0.4" y="0.3" z="0.2">
             <origin xyz="0.2 0 0.1" rpy="0 0 0"/>
         </xacro:inertial_box>
     </link>
-    <!-- Left wheel -->
-    <joint name = "left_wheel_joint" type = "continuous">
-        <parent link = "base link"/>
-        <child link = "left wheel"/>
-        <origin xyz = "0 0.175 0" rpy ="-${pi/2} 0 0"/>
-        <axis xyz = "0 0 1"/>
+    <!-- Rear left wheel -->
+    <joint name="rear_left_wheel_joint" type="continuous">
+        <parent link="base link"/>
+        <child link="rear_left_wheel"/>
+        <origin xyz="0 0.190 0" rpy="${pi/2} 0 0"/>
+        <axis xyz="0 0 1"/>
     </joint>
-    <link name = "left wheel">
+    <link name="rear_left_wheel">
         <visual>
             <geometry>
-                <cylinder radius = "0.1" length = "0.05" />
+                <cylinder radius="0.1" length="0.05" />
             </geometry>
-            <material name = "blue"/>
-        </visual>
-        <collision>
-            <geometry>
-                <cylinder radius = "0.1" length = "0.05" />
-            </geometry>
-        </collision>
-        <xacro:inertial_cylinder mass="0.2" length="0.05" radius="0.1">
-            <origin xyz = "0 0 0" rpy="0 0 0"/>
-        </xacro:inertial_cylinder>
-    </link>
-    <!-- Right wheel -->
-    <joint name = "right_wheel_joint" type = "continuous">
-        <parent link = "base link"/>
-        <child link = "right wheel"/>
-        <origin xyz = "0 -0.175 0" rpy ="${pi/2} 0 0"/>
-        <axis xyz = "0 0 -1"/>
-    </joint>
-    <link name = "right wheel">
-        <visual>
-            <geometry>
-                <cylinder radius = "0.1" length = "0.05" />
-            </geometry>
-            <material name = "blue"/>
+            <material name="blue"/>
         </visual>
         <collision>
@@ -91,25 +68,72 @@
         </xacro:inertial_cylinder>
     </link>
-    <!-- chaster wheel (that bulb like thing) -->
-    <joint name = "chaster_wheel_joint" type = "fixed">
-        <parent link = "base link"/>
-        <child link = "chaster wheel"/>
-        <origin xyz = "0.2 0 0" rpy ="0 0 0"/>
+    <!-- Rear right wheel -->
+    <joint name="rear_right_wheel_joint" type="continuous">
+        <parent link="base link"/>
+        <child link="rear_right_wheel"/>
+        <origin xyz="0 -0.190 0" rpy="${pi/2} 0 0"/>
+        <axis xyz="0 0 -1"/>
     </joint>
-    <link name = "chaster wheel">
+    <link name="rear_right_wheel">
         <visual>
             <geometry>
-                <sphere radius = "0.1"/>
+                <cylinder radius="0.1" length="0.05" />
             </geometry>
-            <material name = "orange"/>
+            <material name="blue"/>
         </visual>
         <collision>
             <geometry>
-                <sphere radius = "0.1"/>
+                <cylinder radius="0.1" length="0.05" />
             </geometry>
         </collision>
-        <xacro:inertial_sphere mass="0.2" radius="0.1">
-            <origin xyz="0 0 0" rpy="0 0 0" />
-        </xacro:inertial_sphere>
+        <xacro:inertial_cylinder mass="0.2" length="0.05" radius="0.1">
+            <origin xyz="0 0 0" rpy="0 0 0"/>
+        </xacro:inertial_cylinder>
+    </link>
+    <!-- Front left wheel -->
+    <joint name="front_left_wheel_joint" type="continuous">
+        <parent link="base link"/>
+        <child link="front_left_wheel"/>
+        <origin xyz="0.23 0.190 0" rpy="${pi/2} 0 0"/>
+        <axis xyz="0 0 1"/>
+    </joint>
+    <link name="front_left_wheel">
+        <visual>
+            <geometry>
+                <cylinder radius="0.1" length="0.05" />
+            </geometry>
+            <material name="blue"/>
+        </visual>
+        <collision>
+            <geometry>
+                <cylinder radius="0.1" length="0.05" />
+            </geometry>
+        </collision>
+        <xacro:inertial_cylinder mass="0.2" length="0.05" radius="0.1">
+            <origin xyz="0 0 0" rpy="0 0 0"/>
+        </xacro:inertial_cylinder>
+    </link>
+    <!-- Front right wheel -->
+    <joint name="front_right_wheel_joint" type="continuous">
+        <parent link="base link"/>
+        <child link="front_right_wheel"/>
+        <origin xyz="0.23 -0.190 0" rpy="${pi/2} 0 0"/>
+        <axis xyz="0 0 -1"/>
+    </joint>
+    <link name="front_right_wheel">
+        <visual>
+            <geometry>
+                <cylinder radius="0.1" length="0.05" />
+            </geometry>
+            <material name="blue"/>
+        </visual>
+        <collision>
+            <geometry>
+                <cylinder radius="0.1" length="0.05" />
+            </geometry>
+        </collision>
+        <xacro:inertial_cylinder mass="0.2" length="0.05" radius="0.1">
+            <origin xyz="0 0 0" rpy="0 0 0"/>
+        </xacro:inertial_cylinder>
     </link>
     <xacro />
