Commit message: updated for 4 wheel robot it works as of now turn moves and stuff

File: src/lidar_robot/description/gazebo_robot_control.xacro (robot description, xacro)
@@ -2,5 +2,5 @@
 <robot xmlns:xacro="http://www.ros.org/wiki/xacro"  name="robot">
     <gazebo>
-        <plugin name="diff_drive" filename="libgazebo_ros_diff_drive.so">
+        <plugin name="diff_drive_back" filename="libgazebo_ros_diff_drive.so">
             <!-- wheel information -->
             <left_joint>rear_left_wheel_joint</left_joint>
@@ -19,4 +19,21 @@
             <publish_wheel_tf>true</publish_wheel_tf>
         </plugin>
+            <plugin name="diff_drive_front" filename="libgazebo_ros_diff_drive.so">
+            <!-- wheel information -->
+            <left_joint>front_left_wheel_joint</left_joint>
+            <right_joint>front_right_wheel_joint</right_joint>
+            <wheel_separation>0.38</wheel_separation>
+            <wheel_diameter>0.2</wheel_diameter>
+            <!-- LIMITS -->
+            <max_wheel_torque>200</max_wheel_torque>
+            <max_wheel_acceleration>10.0</max_wheel_acceleration>
+            <!-- oUTPUT -->
+            <odometry_frame>odom</odometry_frame>
+            <robot_base_frame>base_link</robot_base_frame>
+            <!-- publish odon -->
+            <publish_odom>true</publish_odom>
+            <publish_odom_tf>true</publish_odom_tf>
+            <publish_wheel_tf>true</publish_wheel_tf>
+        </plugin>
     </gazebo>
 </robot>

File: src/lidar_robot/description/robot_core.xacro (robot description, xacro)
@@ -19,9 +19,9 @@
     </material>
     <!-- first link is called as base link -->
-    <link name="base link">
+    <link name="base_link">
     </link>
     <!-- chassis (box with some dimensions) -->
     <joint name="chassis_joint" type="fixed">
-        <parent link="base link"/>
+        <parent link="base_link"/>
         <child link="chassis"/>
         <origin xyz="-0.1 0 0"/>
@@ -47,5 +47,5 @@
     <!-- Rear left wheel -->
     <joint name="rear_left_wheel_joint" type="continuous">
-        <parent link="base link"/>
+        <parent link="base_link"/>
         <child link="rear_left_wheel"/>
         <origin xyz="0 0.190 0" rpy="${pi/2} 0 0"/>
@@ -70,5 +70,5 @@
     <!-- Rear right wheel -->
     <joint name="rear_right_wheel_joint" type="continuous">
-        <parent link="base link"/>
+        <parent link="base_link"/>
         <child link="rear_right_wheel"/>
         <origin xyz="0 -0.190 0" rpy="${pi/2} 0 0"/>
@@ -93,5 +93,5 @@
     <!-- Front left wheel -->
     <joint name="front_left_wheel_joint" type="continuous">
-        <parent link="base link"/>
+        <parent link="base_link"/>
         <child link="front_left_wheel"/>
         <origin xyz="0.23 0.190 0" rpy="${pi/2} 0 0"/>
@@ -116,5 +116,5 @@
     <!-- Front right wheel -->
     <joint name="front_right_wheel_joint" type="continuous">
-        <parent link="base link"/>
+        <parent link="base_link"/>
         <child link="front_right_wheel"/>
         <origin xyz="0.23 -0.190 0" rpy="${pi/2} 0 0"/>
