Commit message: made lidar and updated world file

File: src/lidar_robot/description/lidar.xacro (robot description, xacro)
@@ -1,3 +1,55 @@
 <?xml version="1.0"?>
 <robot xmlns:xacro="http://www.ros.org/wiki/xacro">
+    <joint name="lazer_joint" type="fixed">
+        <origin xyz="0.2 0 0.2" rpy="0.0 0.0 0.0"/>
+        <parent link="chassis"/>
+        <child link="lazer_frame"/>
+        <axis xyz="0.0 0.0 0.0"/>
+        <limit lower="0.0" upper="0.0" effort="0.0" velocity="0.0"/>
+    </joint>
+    <link name="lazer_frame">
+        <visual>
+            <geometry>
+                <cylinder radius="0.05" length="0.25"/>
+            </geometry>
+            <material name="rod">
+                <color rgba="1.0 0.0 0.0 1.0"/>
+            </material>
+        </visual>
+        <collision>
+            <geometry>
+                <cylinder radius="0.2" length="0.25"/>
+            </geometry>
+        </collision>
+        <xacro:inertial_cylinder mass="0.1" radius="0.2" length="0.25">
+            <origin xyz="0.0 0.0 0.0" rpy="0.0 0.0 0.0"/>
+        </xacro:inertial_cylinder>
+    </link>
+    <gazebo reference="lazer_frame">
+        <sensor name="laser" type="ray">
+            <pose> 0 0 0 0 0 0 </pose>
+            <visualize>true</visualize>
+            <update_rate>10</update_rate>
+            <ray>
+                <scan>
+                    <horizontal>
+                        <samples>360</samples>
+                        <min_angle>-3.14</min_angle>
+                        <max_angle>3.14</max_angle>
+                    </horizontal>
+                </scan>
+                <range>
+                    <min>0.3</min>
+                    <max>12</max>
+                </range>
+            </ray>
+            <plugin name="laser_controller" filename="libgazebo_ros_ray_sensor.so">
+                <ros>
+                    <argument>~/out:=scan</argument>
+                </ros>
+                <output_type>sensor_msgs/LaserScan</output_type>
+                <frame_name>lazer_frame</frame_name>
+            </plugin>
+        </sensor>
+    </gazebo>
 </robot>

File: src/lidar_robot/description/robot.urdf.xacro (robot description, xacro)
@@ -5,3 +5,4 @@
     <xacro:include filename="robot_core.xacro" />
     <xacro:include filename="gazebo_robot_control.xacro"/>
+    <xacro:include filename="lidar.xacro"/>
 </robot>
