Commit message: point cloud files added robot updated

File: src/lidar_robot/description/camera.xacro (robot description, xacro)
@@ -36,5 +36,5 @@
             <update_rate>10</update_rate>
             <camera>
-                <horizontal_fov>1.3962634</horizontal_fov> <!-- put actual cam zoom -->
+                <horizontal_fov>1.3962634</horizontal_fov>                <!-- put actual cam zoom -->
                 <image>
                     <width>640</width>

File: src/lidar_robot/description/gazebo_robot_control.xacro (robot description, xacro)
@@ -1,4 +1,4 @@
 <?xml version="1.0"?>
-<robot xmlns:xacro="http://www.ros.org/wiki/xacro"  name="robot">
+<robot xmlns:xacro="http://www.ros.org/wiki/xacro" name="robot">
     <gazebo>
         <plugin name="diff_drive_back" filename="libgazebo_ros_diff_drive.so">

File: src/lidar_robot/description/inertial_macros.xacro (robot description, xacro)
@@ -1,4 +1,4 @@
 <?xml version="1.0"?>
-<robot xmlns:xacro="http://www.ros.org/wiki/xacro" >
+<robot xmlns:xacro="http://www.ros.org/wiki/xacro">
     <!-- Specify some standard inertial calculations https://en.wikipedia.org/wiki/List_of_moments_of_inertia -->
     <!-- These make use of xacro's mathematical functionality -->
@@ -7,7 +7,5 @@
             <xacro:insert_block name="origin"/>
             <mass value="${mass}" />
-            <inertia ixx="${(2/5) * mass * (radius*radius)}" ixy="0.0" ixz="0.0"
-                    iyy="${(2/5) * mass * (radius*radius)}" iyz="0.0"
-                    izz="${(2/5) * mass * (radius*radius)}" />
+            <inertia ixx="${(2/5) * mass * (radius*radius)}" ixy="0.0" ixz="0.0" iyy="${(2/5) * mass * (radius*radius)}" iyz="0.0" izz="${(2/5) * mass * (radius*radius)}" />
         </inertial>
     </xacro:macro>
@@ -16,7 +14,5 @@
             <xacro:insert_block name="origin"/>
             <mass value="${mass}" />
-            <inertia ixx="${(1/12) * mass * (y*y+z*z)}" ixy="0.0" ixz="0.0"
-                    iyy="${(1/12) * mass * (x*x+z*z)}" iyz="0.0"
-                    izz="${(1/12) * mass * (x*x+y*y)}" />
+            <inertia ixx="${(1/12) * mass * (y*y+z*z)}" ixy="0.0" ixz="0.0" iyy="${(1/12) * mass * (x*x+z*z)}" iyz="0.0" izz="${(1/12) * mass * (x*x+y*y)}" />
         </inertial>
     </xacro:macro>
@@ -25,7 +21,5 @@
             <xacro:insert_block name="origin"/>
             <mass value="${mass}" />
-            <inertia ixx="${(1/12) * mass * (3*radius*radius + length*length)}" ixy="0.0" ixz="0.0"
-                    iyy="${(1/12) * mass * (3*radius*radius + length*length)}" iyz="0.0"
-                    izz="${(1/2) * mass * (radius*radius)}" />
+            <inertia ixx="${(1/12) * mass * (3*radius*radius + length*length)}" ixy="0.0" ixz="0.0" iyy="${(1/12) * mass * (3*radius*radius + length*length)}" iyz="0.0" izz="${(1/2) * mass * (radius*radius)}" />
         </inertial>
     </xacro:macro>

File: src/lidar_robot/description/robot.urdf.xacro (robot description, xacro)
@@ -1,4 +1,5 @@
 <?xml version="1.0"?>
-<robot xmlns:xacro="http://www.ros.org/wiki/xacro"  name="robot">
+<robot xmlns:xacro="http://www.ros.org/wiki/xacro" name="robot">
+  <xacro:include filename="$(find velodyne_description)/urdf/VLP-16.urdf.xacro"/>
     <!-- Example link -->
     <!-- <link name="base_link"></link> -->
@@ -7,3 +8,4 @@
     <xacro:include filename="lidar.xacro"/>
     <xacro:include filename="camera.xacro"/>
+    <xacro:include filename="pointcloud.xacro"/>
 </robot>
