Commit message: robot urdf compiled

File: src/lidar_robot/description/robot.urdf (robot description, URDF)
Before this commit: robot robot, 11 links, 10 joints
Links:
- link velodyne: geometry collision sphere radius=0; visual mesh filename=package://velodyne_description/meshes/VLP16_scan.dae
Joints:
- joint velodyne_base_mount_joint: origin xyz=0 0 -0.4 rpy=0 3.141592653589793 0 -> xyz=0.2 0 0.35 rpy=0 3.141592653589793 0; parent base_link -> chassis
